File: main.brd (EAGLE design)
At the start: 80 x 80 mm, 11 parts

Commit message: updated
Parts:
- removed JP3: (no value), pinhead:1X06
- added R1, R2, R3, R4: 10K, rcl:R0603
- added SENSORS: (no value), pinhead:1X06
- renumbered JP1 to LCD1, JP2 to LCD2, JP7 to BAT
Connections:
- new net N$7: R4.1, S4.1, S4.3
- net 3.3V: now also R1.2, R2.2, R3.2, R4.2, SENSORS.6; no longer JP3.6, S1.3, S2.3, S3.3, S4.3
- net GND2: now also SENSORS.5; no longer JP3.5
- net GPIO12: no longer S4.1
- net GPIO26: now also R3.1, S3.3
- net GPIO27: now also R2.1, S2.3
- net GPIO34: now also SENSORS.2; no longer JP3.2
- net GPIO35: now also SENSORS.3; no longer JP3.3
- net GPIO36: now also SENSORS.1; no longer JP3.1
- net GPIO39: now also SENSORS.4; no longer JP3.4
- net GPIO5: now also R1.1, S1.3
Routing:
- net GPIO12: track 34.9 -> 1.18 mm
- net N$7: track 0.00 -> 11.7 mm
- net GPIO26: track 29.5 -> 41.1 mm
- net GPIO27: track 33.8 -> 45.3 mm
- net GPIO5: track 78.6 -> 89.5 mm
- net 3.3V: track 254.8 -> 260.8 mm
- net GPIO35: track 52.7 -> 47.5 mm
- net B+: track 97.3 -> 100.8 mm
- net GND2: track 144.0 -> 146.3 mm, vias 1 -> 3
- net GPIO36: track 65.9 -> 67.7 mm
- net GPIO2: track 35.2 -> 36.5 mm
- net GPIO34: track 41.5 -> 42.4 mm
