File: main.sch (EAGLE design)
At the start: 11 parts

Commit message: updated
Parts:
- removed JP3: (no value), pinhead:PINHD-1X6
- added R1, R2, R3, R4: 10K, rcl:R-US_R0603
- added SENSORS: (no value), pinhead:PINHD-1X6
- renumbered JP1 to LCD1, JP2 to LCD2, JP7 to BAT
Connections:
- new net N$7: R4.1, S41.S, S42.S
- net 3.3V: now also R1.2, R2.2, R3.2, R4.2, SENSORS.6; no longer JP3.6, S12.S, S22.S, S32.S, S42.S
- net GND2: now also SENSORS.5; no longer JP3.5
- net GPIO12: no longer S41.S
- net GPIO26: now also R3.1, S32.S
- net GPIO27: now also R2.1, S22.S
- net GPIO34: now also SENSORS.2; no longer JP3.2
- net GPIO35: now also SENSORS.3; no longer JP3.3
- net GPIO36: now also SENSORS.1; no longer JP3.1
- net GPIO39: now also SENSORS.4; no longer JP3.4
- net GPIO5: now also R1.1, S12.S
Other:
- note added: "TP4056"
