File: sensors.sch (EAGLE design)
At the start: 5 parts

Commit message: updated
Parts:
- added PAD1, PAD10, PAD11, PAD12, PAD2, PAD3, PAD4, PAD5, PAD6, PAD7, PAD8, PAD9: WIREPADSMD1,27-254, wirepad:WIREPADSMD1,27-254
Connections:
- net 3.3V: now also PAD12.P, PAD3.P, PAD6.P, PAD9.P; no longer U$1.VCC, U$2.VCC, U$3.VCC, U$4.VCC
- net GND: now also PAD11.P, PAD2.P, PAD5.P, PAD8.P; no longer U$1.GND, U$2.GND, U$3.GND, U$4.GND
- net GPIO34: now also PAD4.P; no longer U$2.A
- net GPIO35: now also PAD7.P; no longer U$3.A
- net GPIO36: now also PAD1.P; no longer U$1.A
- net GPIO39: now also PAD10.P; no longer U$4.A
Other:
- moved on the sheet: JP1
